File: PCB/DualSlopeADC.kicad_pcb (KiCad board)
At the start: 2 copper layers, 65 x 56.5 mm, 15 parts, among them J1 RPi_GPIO, J5 Conn_01x02, J6 Conn_01x02, J7 Conn_01x02, U1 OPA1692xDGK, U2 OPA1692xDGK, U3 OPA1692xDGK

Commit message: .
Parts:
- removed C1: C, Capacitor_SMD:C_0805_2012Metric
- removed J1: RPi_GPIO, RPI_Hat:RPI_Hat_B+
- removed J5, J6, J7: Conn_01x02, Connector_PinHeader_2.54mm:PinHeader_1x02_P2.54mm_Vertical
- removed R1, R2, R3, R4, R5, R6, R7: R, Resistor_SMD:R_0603_1608Metric
- added U4: ADG419BRM, Package_SO:MSOP-8_3x3mm_P0.65mm, F.Cu at (134.4, 87.5)
- added U5: LTC6752xSC6-4, Package_TO_SOT_SMD:SOT-363_SC-70-6, F.Cu at (132.8, 91.7)
- added U6: CA56-12EWA, Display_7Segment:CA56-12EWA, F.Cu at (65.8, 76.4)
- added U8: 74HC595, Package_DIP:DIP-16_W7.62mm, F.Cu at (93.2, 46.1)
- U1: value OPA1692xDGK -> CH32V003FxPx; footprint Package_SO:VSSOP-8_3x3mm_P0.65mm -> Package_SO:TSSOP-20_4.4x6.5mm_P0.65mm
- U2: value OPA1692xDGK -> ADR4533; footprint Package_SO:VSSOP-8_3x3mm_P0.65mm -> Package_SO:SOIC-8_3.9x4.9mm_P1.27mm
- U3: value OPA1692xDGK -> AD8606ARZ; footprint Package_SO:VSSOP-8_3x3mm_P0.65mm -> Package_SO:SOIC-8_3.9x4.9mm_P1.27mm
- moved U2 18.7 mm to (126.4, 80.4)
- moved U3 17.7 mm to (126.4, 87.0)
- moved U1 8.34 mm to (135.4, 81.1)
Connections:
- U1 pad 1: Net-(U1A--) -> unconnected-(U1-PD4-Pad1)
- U1 pad 2: Net-(U1A--) -> unconnected-(U1-PD5-Pad2)
- U1 pad 3: Net-(Q1-D) -> unconnected-(U1-PD6-Pad3)
- U1 pad 4: (no net) -> unconnected-(U1-PD7-Pad4)
- U1 pad 5: (no net) -> unconnected-(U1-PA1-Pad5)
- U1 pad 6: (no net) -> unconnected-(U1-PA2-Pad6)
- U1 pad 7: (no net) -> unconnected-(U1-VSS-Pad7)
- U1 pad 8: (no net) -> unconnected-(U1-PD0-Pad8)
- U2 pad 1: Net-(U3A--) -> unconnected-(U2-NC-Pad1)
- U2 pad 2: Net-(U2A--) -> unconnected-(U2-IN-Pad2)
- U2 pad 3: GND -> unconnected-(U2-NC-Pad3)
- U2 pad 4: (no net) -> unconnected-(U2-GND-Pad4)
- U2 pad 5: (no net) -> unconnected-(U2-NC-Pad5)
- U2 pad 6: (no net) -> unconnected-(U2-OUT-Pad6)
- U2 pad 7: (no net) -> unconnected-(U2-NC-Pad7)
- U2 pad 8: (no net) -> unconnected-(U2-NC-Pad8)
- U3 pad 1: Net-(J1-BCM17) -> unconnected-(U3-Pad1)
- U3 pad 2: Net-(U3A--) -> unconnected-(U3A---Pad2)
- U3 pad 3: GND -> unconnected-(U3A-+-Pad3)
Other:
- board outline removed

Commit message: PCB design anfang
Parts:
- added C2: 0.1u, Capacitor_SMD:C_0805_2012Metric, F.Cu at (157.3, 90.9)
- added C3: 0.1u, Capacitor_SMD:C_0805_2012Metric, F.Cu at (157.3, 93.9)
- added C4: 1m, Capacitor_SMD:C_0805_2012Metric, F.Cu at (157.3, 97.0)
- added C5: 130p, Capacitor_SMD:C_0805_2012Metric, F.Cu at (157.3, 100.0)
- added C6: 100u, Capacitor_THT:CP_Radial_D12.5mm_P5.00mm, F.Cu at (149.2, 73.7)
- added J1: Conn_01x02_Pin, Connector_PinHeader_2.54mm:PinHeader_1x02_P2.54mm_Vertical, F.Cu at (146.6, 61.8)
- added J3: Conn_01x02_Pin, Connector_PinHeader_2.54mm:PinHeader_1x02_P2.54mm_Vertical, F.Cu at (151.2, 61.8)
- added J4: Conn_01x02_Pin, Connector_PinHeader_2.54mm:PinHeader_1x02_P2.54mm_Vertical, F.Cu at (155.8, 61.8)
- added J5: Conn_01x02_Pin, Connector_PinHeader_2.54mm:PinHeader_1x02_P2.54mm_Vertical, F.Cu at (160.4, 61.8)
- added R1: 1k, Resistor_SMD:R_0603_1608Metric, F.Cu at (160.7, 71.8)
- added R2: 10Meg, Resistor_SMD:R_0603_1608Metric, F.Cu at (160.7, 74.3)
- added R3: 100k, Resistor_SMD:R_0603_1608Metric, F.Cu at (160.7, 76.8)
- U3: value AD8606ARZ -> AD8605ARTZ-R2; footprint Package_SO:SOIC-8_3.9x4.9mm_P1.27mm -> footprints:SOT95P290X145-5N
- moved U8 64.2 mm to (145.9, 82.7)
- moved U6 60.7 mm to (126.4, 79.1)
- moved U2 40.3 mm to (157.6, 105.9)
- moved U5 36.3 mm to (160.8, 68.6)
- moved U3 31.1 mm to (157.5, 87.4)
- moved U1 28.9 mm to (149.0, 106.6)
- moved U4 24.8 mm to (158.8, 83.0)
Connections:
- U1 pad 4: unconnected-(U1-PD7-Pad4) -> /RESET
- U1 pad 7: unconnected-(U1-VSS-Pad7) -> GND
- U1 pad 9: unconnected-(U1-VDD-Pad9) -> VCC_5V
- U2 pad 2: unconnected-(U2-IN-Pad2) -> VCC_5V
- U2 pad 4: unconnected-(U2-GND-Pad4) -> GND
- U2 pad 6: unconnected-(U2-OUT-Pad6) -> Net-(J1-Pin_1)
- U3 pad 1: unconnected-(U3-Pad1) -> Net-(U3-OUTA)
- U3 pad 2: unconnected-(U3A---Pad2) -> GND
- U3 pad 3: unconnected-(U3A-+-Pad3) -> VCC_3V3
- U3 pad 4: (no net) -> Net-(U3--INA)
- U3 pad 5: (no net) -> VCC_5V
- U4 pad 1: unconnected-(U4-Pad1) -> Net-(R3-Pad1)
- U4 pad 2: unconnected-(U4-Pad2) -> Net-(C4-Pad1)
- U4 pad 3: (no net) -> GND
- U4 pad 4: (no net) -> VCC_5V
- U4 pad 5: (no net) -> VCC_5V
- U4 pad 6: unconnected-(U4-Pad6) -> /GPIO_Control
- U4 pad 7: (no net) -> GND
- U4 pad 8: unconnected-(U4-Pad8) -> VCC_5V
- U5 pad 1: unconnected-(U5-Pad1) -> /GPIO_Input
- U5 pad 2: unconnected-(U5-VEE-Pad2) -> GND
- U5 pad 3: unconnected-(U5-+-Pad3) -> VCC_3V3
- U5 pad 4: unconnected-(U5---Pad4) -> Net-(U3-OUTA)
- U5 pad 5: unconnected-(U5-VDD-Pad5) -> VCC_5V
- U5 pad 6: unconnected-(U5-VCC-Pad6) -> VCC_5V

Commit message: CH32fun integriert
Parts:
- moved U6 66.8 mm to (153.8, 139.9), turned to 90 degrees
- moved U2 40.3 mm to (187.0, 78.3)
- moved U1 38.9 mm to (187.9, 105.5)
- moved J5 25.7 mm to (185.5, 56.1)
- moved J4 15.1 mm to (161.5, 47.8)
- moved J1 11.1 mm to (136.0, 58.3)
- moved J3 8.59 mm to (147.6, 54.0)
Changed lines of the file:
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@@
 	(footprint "Connector_PinHeader_2.54mm:PinHeader_1x02_P2.54mm_Vertical"
 		(layer "F.Cu")
-		(at 160.355 61.79)
+		(at 185.46 56.12)
 		(descr "Through hole straight pin header, 1x02, 2.54mm pitch, single row")
 		(tags "Through hole pin header THT 1x02 2.54mm single row")
@@
 	(footprint "Package_SO:SOIC-8_3.9x4.9mm_P1.27mm"
 		(layer "F.Cu")
-		(at 157.635 105.91)
+		(at 187.03 78.31)
 		(descr "SOIC, 8 Pin (JEDEC MS-012AA, https://www.analog.com/media/en/package-pcb-resources/package/pkg_pdf/soic_narrow-r/r_8.pdf), generated with kicad-footprint-generator ipc_gullwing_generator.py")
 		(tags "SOIC SO")
@@
 	(footprint "Connector_PinHeader_2.54mm:PinHeader_1x02_P2.54mm_Vertical"
 		(layer "F.Cu")
-		(at 155.765 61.79)
+		(at 161.47 47.83)
 		(descr "Through hole straight pin header, 1x02, 2.54mm pitch, single row")
 		(tags "Through hole pin header THT 1x02 2.54mm single row")
@@
 	(footprint "Connector_PinHeader_2.54mm:PinHeader_1x02_P2.54mm_Vertical"
 		(layer "F.Cu")
-		(at 151.175 61.79)
+		(at 147.57 53.99)
 		(descr "Through hole straight pin header, 1x02, 2.54mm pitch, single row")
 		(tags "Through hole pin header THT 1x02 2.54mm single row")
@@
 	(footprint "Package_SO:TSSOP-20_4.4x6.5mm_P0.65mm"
 		(layer "F.Cu")
-		(at 149.04 106.58)
+		(at 187.93 105.55)
 		(descr "TSSOP, 20 Pin (JEDEC MO-153 Var AC https://www.jedec.org/document_search?search_api_views_fulltext=MO-153), generated with kicad-footprint-generator ipc_gullwing_generator.py")
 		(tags "TSSOP SO")
@@
 	(footprint "Connector_PinHeader_2.54mm:PinHeader_1x02_P2.54mm_Vertical"
 		(layer "F.Cu")
-		(at 146.585 61.79)
+		(at 136.03 58.315)
 		(descr "Through hole straight pin header, 1x02, 2.54mm pitch, single row")
 		(tags "Through hole pin header THT 1x02 2.54mm single row")
@@
 	(footprint "Display_7Segment:CA56-12EWA"
 		(layer "F.Cu")
-		(at 126.4 79.07)
+		(at 153.8 139.94 90)
 		(descr "4 digit 7 segment green LED, http://www.kingbrightusa.com/images/catalog/SPEC/CA56-12EWA.pdf")
 		(tags "4 digit 7 segment green LED")
 		(property "Reference" "U6"
-			(at -0.4 -20.31 0)
+			(at -0.4 -20.31 90)
 			(layer "F.SilkS")
 			(effects
@@
 		)
 		(property "Value" "CA56-12EWA"
-			(at 2.37 33.21 0)
+			(at 2.37 33.21 90)
 			(layer "F.Fab")
 			(effects
@@
 		)
 		(property "Datasheet" "http://www.kingbrightusa.com/images/catalog/SPEC/CA56-12EWA.pdf"
-			(at 0 0 0)
+			(at 0 0 90)
 			(unlocked yes)
 			(layer "F.Fab")
@@
 		)
 		(property "Description" "4 digit 7 segment high efficiency red LED, common anode"
-			(at 0 0 0)
+			(at 0 0 90)
 			(unlocked yes)
 			(layer "F.Fab")
@@
 		(attr through_hole)
 		(fp_line
-			(start -2.38 -1)
-			(end -2.38 1)
+			(start -2 -18.92)
+			(end 17.24 -18.92)
 			(stroke
 				(width 0.12)
@@
 		)
 		(fp_line
-			(start -2 -18.92)
-			(end 17.24 -18.92)
+			(start -2.38 -1)
+			(end -2.38 1)
 			(stroke
 				(width 0.12)
@@
 		)
 		(fp_line
-			(start -2 31.62)
-			(end 17.24 31.62)
+			(start 17.24 31.62)
+			(end 17.24 -18.92)
 			(stroke
 				(width 0.12)
@@
 		)
 		(fp_line
-			(start 17.24 31.62)
-			(end 17.24 -18.92)
+			(start -2 31.62)
+			(end 17.24 31.62)
 			(stroke
 				(width 0.12)
@@
 		)
 		(fp_line
-			(start -2.13 -19.05)
-			(end 17.37 -19.05)
+			(start 17.37 -19.05)
+			(end 17.37 31.75)
 			(stroke
 				(width 0.05)
@@
 		)
 		(fp_line
-			(start -2.13 31.75)
-			(end -2.13 -19.05)
+			(start -2.13 -19.05)
+			(end 17.37 -19.05)
 			(stroke
 				(width 0.05)
@@
 		)
 		(fp_line
-			(start 17.37 -19.05)
-			(end 17.37 31.75)
+			(start 17.37 31.75)
+			(end -2.13 31.75)
 			(stroke
 				(width 0.05)
@@
 		)
 		(fp_line
-			(start 17.37 31.75)
-			(end -2.13 31.75)
+			(start -2.13 31.75)
+			(end -2.13 -19.05)
 			(stroke
 				(width 0.05)
@@
 		)
 		(fp_line
-			(start -1.88 -18.8)
-			(end 17.12 -18.8)
+			(start 17.12 -18.8)
+			(end 17.12 31.5)
 			(stroke
 				(width 0.1)
@@
 		)
 		(fp_line
-			(start -1.88 -1)
-			(end -1.88 -18.8)
+			(start -1.88 -18.8)
+			(end 17.12 -18.8)
 			(stroke
 				(width 0.1)
@@
 		)
 		(fp_line
-			(start -1.88 1)
-			(end -1.88 31.5)
+			(start -1.88 -1)
+			(end -1.88 -18.8)
 			(stroke
 				(width 0.1)
@@
 		)
 		(fp_line
-			(start -1.88 1)
-			(end -0.88 0)
+			(start -0.88 0)
+			(end -1.88 -1)
 			(stroke
 				(width 0.1)
@@
 		)
 		(fp_line
-			(start -1.88 31.5)
-			(end 17.12 31.5)
+			(start -1.88 1)
+			(end -0.88 0)
 			(stroke
 				(width 0.1)
@@
 		)
 		(fp_line
-			(start -0.88 0)
-			(end -1.88 -1)
+			(start -1.88 1)
+			(end -1.88 31.5)
 			(stroke
 				(width 0.1)
@@
 		)
 		(fp_line
-			(start 17.12 -18.8)
+			(start -1.88 31.5)
 			(end 17.12 31.5)
 			(stroke
@@
 		)
 		(fp_text user "${REFERENCE}"
-			(at 8.128 6.604 0)
+			(at 8.128 6.604 90)
 			(layer "F.Fab")
 			(effects
@@
 		)
 		(pad "1" thru_hole rect
-			(at 0 0)
+			(at 0 0 90)
 			(size 1.5 1.5)
 			(drill 1)
@@
 		)
 		(pad "2" thru_hole circle
-			(at 0 2.54)
+			(at 0 2.54 90)
 			(size 1.5 1.5)
 			(drill 1)
@@
 		)
 		(pad "3" thru_hole circle
-			(at 0 5.08)
+			(at 0 5.08 90)
 			(size 1.5 1.5)
 			(drill 1)
@@
 		)
 		(pad "4" thru_hole circle
-			(at 0 7.62)
+			(at 0 7.62 90)
 			(size 1.5 1.5)
 			(drill 1)
@@
 		)
 		(pad "5" thru_hole circle
-			(at 0 10.16)
+			(at 0 10.16 90)
 			(size 1.5 1.5)
 			(drill 1)
@@
 		)
 		(pad "6" thru_hole circle
-			(at 0 12.7)
+			(at 0 12.7 90)
 			(size 1.5 1.5)
 			(drill 1)
@@
 		)
 		(pad "7" thru_hole circle
-			(at 15.24 12.7)
+			(at 15.24 12.7 90)
 			(size 1.5 1.5)
 			(drill 1)
@@
 		)
 		(pad "8" thru_hole circle
-			(at 15.24 10.16)
+			(at 15.24 10.16 90)
 			(size 1.5 1.5)
 			(drill 1)
@@
 		)
 		(pad "9" thru_hole circle
-			(at 15.24 7.62)
+			(at 15.24 7.62 90)
 			(size 1.5 1.5)
 			(drill 1)
@@
 		)
 		(pad "10" thru_hole circle
-			(at 15.24 5.08)
+			(at 15.24 5.08 90)
 			(size 1.5 1.5)
 			(drill 1)
@@
 		)
 		(pad "11" thru_hole circle
-			(at 15.24 2.54)
+			(at 15.24 2.54 90)
 			(size 1.5 1.5)
 			(drill 1)
@@
 		)
 		(pad "12" thru_hole circle
-			(at 15.24 0)
+			(at 15.24 0 90)
 			(size 1.5 1.5)
 			(drill 1)

Commit message: pcb weiter
Parts:
- removed R1: 1k, Resistor_SMD:R_0603_1608Metric
- removed U8: 74HC595, Package_DIP:DIP-16_W7.62mm
- added J2: Conn_01x02_Pin, Connector_PinHeader_2.54mm:PinHeader_1x02_P2.54mm_Vertical, F.Cu at (188.5, 132.6)
- added J6: Conn_01x02_Pin, Connector_PinHeader_2.54mm:PinHeader_1x02_P2.54mm_Vertical, F.Cu at (188.3, 118.0)
- added J7: Conn_01x02_Pin, Connector_PinHeader_2.54mm:PinHeader_1x02_P2.54mm_Vertical, F.Cu at (190.9, 122.6)
- added R4: 330, Resistor_SMD:R_0603_1608Metric, F.Cu at (196.7, 100.8)
- added R5: 330, Resistor_SMD:R_0603_1608Metric, F.Cu at (200.0, 100.8)
- added R6: 330, Resistor_SMD:R_0603_1608Metric, F.Cu at (202.0, 100.8)
- added R7: 330, Resistor_SMD:R_0603_1608Metric, F.Cu at (192.1, 100.8)
- C4: value 1m -> 0.1u
- U6: footprint Display_7Segment:CA56-12EWA -> 3461BS_4Digit_7SegDisplay:3461BS_4Digit_7SegDisplay
- moved J4 101.7 mm to (198.5, 142.6), turned to -90 degrees
- moved J3 90.0 mm to (201.7, 125.9), turned to 90 degrees
- moved J1 84.2 mm to (168.4, 136.0), turned to 180 degrees
- moved J5 82.0 mm to (188.4, 138.1), turned to 90 degrees
- moved U6 72.1 mm to (196.8, 82.1), turned to -90 degrees
- moved U5 66.7 mm to (196.6, 125.0), turned to -90 degrees
- moved R3 65.9 mm to (201.1, 128.9), turned to 180 degrees
- moved U2 62.6 mm to (161.1, 135.3)
- moved C6 61.4 mm to (142.6, 134.7), turned to -90 degrees
- moved U3 60.6 mm to (197.6, 132.9), turned to 90 degrees
- moved C3 59.5 mm to (197.5, 137.8), turned to 180 degrees
- moved U4 55.6 mm to (203.8, 115.6), turned to 180 degrees
- moved C5 48.8 mm to (196.6, 128.9), turned to 180 degrees
- moved C2 44.9 mm to (153.2, 135.7), turned to -90 degrees
- moved C4 44.1 mm to (189.9, 126.6)
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Connections:
- C4 pad 1: Net-(C4-Pad1) -> GND
- C4 pad 2: GND -> NRST
- R2 pad 1: Vin -> GND
- R2 pad 2: VCC_3V3 -> Vin
- U1 pad 1: unconnected-(U1-PD4-Pad1) -> Net-(U1-PD4)
- U1 pad 10: unconnected-(U1-PC0-Pad10) -> DIG_B
- U1 pad 11: unconnected-(U1-PC1-Pad11) -> Net-(U1-PC1)
- U1 pad 12: unconnected-(U1-PC2-Pad12) -> Net-(U1-PC2)
- U1 pad 13: unconnected-(U1-PC3-Pad13) -> DIG_F
- U1 pad 14: unconnected-(U1-PC4-Pad14) -> DIG_A
- U1 pad 15: unconnected-(U1-PC5-Pad15) -> Net-(U1-PC5)
- U1 pad 16: unconnected-(U1-PC6-Pad16) -> DIG_E
- U1 pad 17: unconnected-(U1-PC7-Pad17) -> DIG_D
- U1 pad 18: unconnected-(U1-PD1-Pad18) -> SWIO
- U1 pad 19: unconnected-(U1-PD2-Pad19) -> DIG_C
- U1 pad 2: unconnected-(U1-PD5-Pad2) -> Tx
- U1 pad 20: unconnected-(U1-PD3-Pad20) -> DIG_G
- U1 pad 3: unconnected-(U1-PD6-Pad3) -> Rx
- U1 pad 4: /RESET -> NRST
- U1 pad 5: unconnected-(U1-PA1-Pad5) -> COMP_OUT
- U1 pad 6: unconnected-(U1-PA2-Pad6) -> COMP_OUT
- U1 pad 8: unconnected-(U1-PD0-Pad8) -> ADC_Control
- U4 pad 2: Net-(C4-Pad1) -> Net-(J2-Pin_2)
- U4 pad 6: /GPIO_Control -> ADC_Control
- U5 pad 1: /GPIO_Input -> COMP_OUT
- U6 pad 1: unconnected-(U6-e-Pad1) -> DIG_E
- U6 pad 10: unconnected-(U6-f-Pad10) -> DIG_F
- U6 pad 11: unconnected-(U6-a-Pad11) -> DIG_A
- U6 pad 12: unconnected-(U6-CA1-Pad12) -> DIG_12
- U6 pad 2: unconnected-(U6-d-Pad2) -> DIG_D
- U6 pad 4: unconnected-(U6-c-Pad4) -> DIG_C
- U6 pad 5: unconnected-(U6-g-Pad5) -> DIG_G
- U6 pad 6: unconnected-(U6-CA4-Pad6) -> DIG_6
- U6 pad 7: unconnected-(U6-b-Pad7) -> DIG_B
- U6 pad 8: unconnected-(U6-CA3-Pad8) -> DIG_8
- U6 pad 9: unconnected-(U6-CA2-Pad9) -> DIG_9
Routing:
- net VCC_5V: track 0.00 -> 48.4 mm
- net DIG_E: track 0.00 -> 33.0 mm
- net DIG_D: track 0.00 -> 30.2 mm
- net DIG_A: track 0.00 -> 29.1 mm
- net DIG_12: track 0.00 -> 26.4 mm
- net DIG_F: track 0.00 -> 26.1 mm
- net DIG_B: track 0.00 -> 24.9 mm
- net DIG_C: track 0.00 -> 24.6 mm
- net DIG_G: track 0.00 -> 21.8 mm
- net DIG_9: track 0.00 -> 17.9 mm
- net NRST: track 0.00 -> 17.4 mm
- net DIG_8: track 0.00 -> 16.1 mm
- net COMP_OUT: track 0.00 -> 13.3 mm
- net DIG_6: track 0.00 -> 11.7 mm
- net Net-(U1-PD4): track 0.00 -> 10.5 mm
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- added copper zone on F.Cu, net GND

Commit message: schaltpan fertig ohne Spannungsfolger
Parts:
- moved C6 89.9 mm to (215.2, 81.5), turned to 180 degrees
- moved R2 86.5 mm to (212.3, 123.2)
- moved C2 75.1 mm to (214.3, 91.9), turned to 180 degrees
- moved U2 65.6 mm to (214.6, 97.3), turned to -90 degrees
- moved J1 56.0 mm to (214.0, 103.6), turned to 90 degrees
- moved J4 39.3 mm to (216.6, 107.6)
- moved J3 38.7 mm to (220.1, 91.9), turned to 180 degrees
- moved C3 32.1 mm to (215.7, 111.2)
- moved J5 30.7 mm to (213.1, 119.9), turned to -90 degrees
- moved J2 29.7 mm to (213.1, 115.9), turned to -90 degrees
- moved R3 4.98 mm to (202.8, 124.2)
- moved U5 4.98 mm to (198.2, 120.2)
- moved U3 4.98 mm to (199.2, 128.2)
- moved C5 4.98 mm to (198.2, 124.2)
Routing:
- net VCC_3V3: track 8.55 -> 48.0 mm
- net VCC_5V: track 48.4 -> 79.5 mm, vias 0 -> 2
- net Net-(R3-Pad1): track 0.00 -> 8.57 mm
- net Vin: track 0.00 -> 7.32 mm
- net GND: track 3.51 -> 10.6 mm, vias 0 -> 1
- net Net-(J2-Pin_2): track 0.00 -> 4.63 mm
- net COMP_OUT: track 13.3 -> 9.33 mm
- net Net-(J1-Pin_1): track 4.81 -> 3.91 mm
- added copper zone on B.Cu, net GND
Other:
- board outline added: 45 x 72 mm

Commit message: Software inm Mounriver studio
Parts:
- added J8: Conn_01x02_Pin, Connector_PinHeader_2.54mm:PinHeader_1x02_P2.54mm_Vertical, F.Cu at (213.1, 119.8)
- moved R2 10.7 mm to (212.2, 112.5)
- moved R3 5.43 mm to (205.9, 119.8), turned to -90 degrees
- moved J5 3.88 mm to (213.1, 123.8)
- moved U3 3.11 mm to (196.9, 126.0)
- moved U5 3.11 mm to (196.0, 118.1)
- moved C5 3.01 mm to (196.0, 122.2)
- moved C4 2.82 mm to (188.1, 124.5)
- moved J7 2.82 mm to (189.0, 120.5)
- moved J6 2.39 mm to (186.5, 116.5)
- moved C3 1.94 mm to (217.6, 111.4), turned to 0 degrees
Connections:
- U1 pad 6: COMP_OUT -> Net-(J8-Pin_2)
Routing:
- net Net-(J8-Pin_2): track 0.00 -> 20.1 mm
- net VCC_3V3: track 48.0 -> 59.5 mm
- net Net-(R3-Pad1): track 8.57 -> 2.36 mm
- net Net-(U3--INA): track 5.89 -> 12.1 mm
- net Vin: track 7.32 -> 11.3 mm
- net COMP_OUT: track 9.33 -> 5.90 mm
- net VCC_5V: track 79.5 -> 76.2 mm
- net NRST: track 17.4 -> 16.1 mm
- net Tx: track 9.61 -> 10.8 mm
- net GND: track 10.6 -> 10.7 mm, vias 1 -> 2

Commit message: platine fertig
Parts:
- removed J1, J4: Conn_01x02_Pin, Connector_PinHeader_2.54mm:PinHeader_1x02_P2.54mm_Vertical
- added J9: Conn_01x02_Pin, Connector_PinHeader_2.54mm:PinHeader_1x02_P2.54mm_Vertical, F.Cu at (186.5, 125.7)
- added U7: AD8656, Package_SO:SOIC-8_3.9x4.9mm_P1.27mm, F.Cu at (214.1, 109.3)
- moved J3 37.0 mm to (214.7, 128.4), turned to 90 degrees
- moved C2 32.4 mm to (214.7, 124.3), turned to 90 degrees
- moved U2 31.4 mm to (207.3, 127.8), turned to 180 degrees
- moved C3 24.1 mm to (200.2, 128.2), turned to -90 degrees
- moved C6 17.6 mm to (215.5, 99.1), turned to 90 degrees
- moved J5 15.5 mm to (219.9, 109.9), turned to 180 degrees
- moved R7 7.66 mm to (192.1, 108.5)
- moved J2 5.24 mm to (216.6, 119.8)
- moved J8 5.24 mm to (216.6, 116.0)
- moved C4 4.98 mm to (192.1, 121.5), turned to 90 degrees
- moved R2 4.28 mm to (208.9, 115.1), turned to -90 degrees
Connections:
- J2 pad 1: Vin -> Net-(J2-Pin_1)
- J2 pad 2: Net-(J2-Pin_2) -> ADC_IN_MC
- J8 pad 1: Vin -> Net-(J2-Pin_1)
- J8 pad 2: Net-(J8-Pin_2) -> ADC_IN_EXT
- R2 pad 2: Vin -> ADC_IN_EXT
- U1 pad 6: Net-(J8-Pin_2) -> ADC_IN_MC
- U2 pad 6: Net-(J1-Pin_1) -> VCC_3V3
- U4 pad 2: Net-(J2-Pin_2) -> ADC_IN_EXT
Routing:
- net VCC_3V3: track 59.5 -> 30.0 mm
- net SWIO: track 0.00 -> 27.5 mm
- net ADC_IN_MC: track 0.00 -> 23.3 mm
- net Net-(J8-Pin_2): track 20.1 -> 0.00 mm
- net VCC_5V: track 76.2 -> 94.3 mm
- net Net-(J2-Pin_1): track 0.00 -> 15.2 mm
- net ADC_IN_EXT: track 0.00 -> 8.18 mm
- net Vin: track 11.3 -> 3.41 mm
- net Net-(U1-PD4): track 10.5 -> 2.87 mm
- net DIG_6: track 11.7 -> 19.4 mm
- net Net-(J2-Pin_2): track 4.63 -> 0.00 mm
- net Net-(J1-Pin_1): track 3.91 -> 0.00 mm
- net GND: track 10.7 -> 11.7 mm, vias 2 -> 4
- net NRST: track 16.1 -> 15.1 mm
- net Tx: track 10.8 -> 11.6 mm
Other:
- board size 45 x 72 mm -> 43 x 69.9 mm
