File: PCB/DualSlopeADC.kicad_sch (KiCad schematic)
At the start: 25 parts, among them J2 Conn_01x02_Pin, J3 Conn_01x02_Pin, J5 Conn_01x02_Pin, J6 Conn_01x02_Pin, J7 Conn_01x02_Pin, J8 Conn_01x02_Pin, J9 Conn_01x02_Pin, U1 CH32V003FxPx, U2 ADR4533, U3 AD8605ARTZ-R2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

Commit message: visulle sachen
Other:
- moved on the sheet: C2, C3, C6, J2, J8, U1, U2, U4B, U6, U7A, U7B, U7C
